Commit message: found fix for joint 'door_hinge' not found in model 'lumi'

File: launch/mikko testing/test.urdf (robot description, URDF)
Before this commit: robot lumi, 13 links, 12 joints
Links:
- added link door; collision mesh filename=package://lumi_description/meshes/door_v4_bin.stl scale=.001 .001 .001; visual mesh filename=package://lumi_description/meshes/door_v4_bin.stl scale=.001 .001 .001
- link base_link: geometry 
Joints:
- added joint door_hinge: type fixed, parent base_link, child door, origin xyz=262 49 0 rpy=0 0 0
