Commit message: fixed all the joint not found errors, roslaunch test2.launch for a working example

File: model/robots/test.urdf (robot description, URDF)
Before this commit: robot lumi, 23 links, 22 joints
Links:
- removed link door_base
- removed link frame_bottom
- removed link frame_left
- removed link frame_left_front
- removed link frame_right
- removed link frame_top
- removed link handle_beam
- removed link handle_core
- removed link handle_latch
- link door: geometry collision mesh filename=package://franka_sim/model/meshes/door_v4_bin.stl scale=.001 .001 .001; visual mesh filename=package://franka_sim/model/meshes/door_v4_bin.stl scale=.001 .001 .001
Joints:
- removed joint door_base_joint
- removed joint frame_bottom_joint
- removed joint frame_left_front_joint
- removed joint frame_left_joint
- removed joint frame_right_joint
- removed joint frame_top_joint
- removed joint handle_beam_joint
- removed joint handle_core
- removed joint handle_latch_joint
- joint door_hinge: origin xyz=0.005 0.005 0.005 rpy=0 0 0 -> xyz=262 49 0 rpy=0 0 0; parent door_base -> base_link
- joint lumi_joint_base_link: origin xyz=0.2 0.2 0.0 rpy=0 0 0 -> xyz=-0.4 0.15 0. rpy=0 0 0
