Commit message: robot and door aligned in rviz and mujoco

File: model/robots/hand.xacro (robot description, xacro)
@@ -28,8 +28,6 @@
       </visual>
       <collision>
-        <origin xyz="0 0.0125 0.028"/>
         <geometry>
-          <box size="0.021 0.025 0.056"/>
-          <!--<mesh filename="package://franka_description/meshes/collision/finger.stl"/>-->
+          <mesh filename="package://franka_description/meshes/collision/finger.stl"/>
         </geometry>
       </collision>
@@ -43,9 +41,7 @@
       </visual>
       <collision>
-        <!--<origin xyz="0 0 0" rpy="0 0 ${pi}"/>-->
-        <origin xyz="0 -0.0125 0.028"/>
+        <origin xyz="0 0 0" rpy="0 0 ${pi}"/>
         <geometry>
-          <box size="0.021 0.025 0.056"/>
-          <!--<mesh filename="package://franka_description/meshes/collision/finger.stl"/>-->
+          <mesh filename="package://franka_description/meshes/collision/finger.stl"/>
         </geometry>
       </collision>

File: model/robots/robot_door.urdf.xacro (robot description, xacro)
@@ -1,6 +1,8 @@
 <?xml version="1.0"?>
 <robot name="lumi" xmlns:xacro="http://www.ros.org/wiki/xacro">
-    <xacro:include filename="$(find franka_description)/robots/panda_arm.xacro"/>
-    <xacro:include filename="$(find franka_description)/robots/hand.xacro"/>
+    <xacro:include filename="$(find franka_sim)/model/robots/panda_arm.xacro"/>
+    <xacro:include filename="$(find franka_sim)/model/robots/hand.xacro"/>
+    <xacro:panda_arm connected_to="base_link" arm_id="lumi" xyz="-0.4 0.15 0.0"/>
+    <xacro:hand ns="lumi" rpy="0 0 ${-pi/4}" connected_to="lumi_link8"/>
     <mujoco>
         <compiler meshdir="../meshes/" balanceinertia="true" discardvisual="false"/>
@@ -10,5 +12,5 @@
     <joint name="door_base_joint" type="fixed">
         <!-- <origin xyz="0.0 0.0 0.052" rpy="0 0 ${pi}"/> -->
-        <origin xyz="0.0 0.0 0.0" rpy="0 0 0"/>
+        <origin xyz="0.4 0.25 0.052" rpy="0 0 ${-pi/2}"/>
         <parent link="base_link"/>
         <child link="door_base"/>
@@ -28,5 +30,5 @@
     <joint name="door_hinge" type="revolute">
         <origin xyz="0.005 0.005 0.005" rpy="0 0 0"/>
-        <limit lower="0" upper="90" effort="10" velocity="10"/>
+        <limit lower="0" upper="${pi/2}" effort="10" velocity="10"/>
         <parent link="door_base"/>
         <child link="door"/>
@@ -46,5 +48,5 @@
     <joint name="handle_core" type="revolute">
         <origin xyz="0.052 -0.06 0.095" rpy="0 0 0"/>
-        <limit lower="0" upper="90" effort="10" velocity="10"/>
+        <limit lower="0" upper="${pi/6}" effort="10" velocity="10"/>
         <parent link="door"/>
         <child link="handle_core"/>
@@ -169,6 +171,4 @@
         <child link="frame_top"/>
     </joint>
-    <xacro:panda_arm connected_to="base_link" arm_id="lumi" xyz="0.2 0.2 0.0"/>
-    <xacro:hand ns="lumi" rpy="0 0 ${-pi/4}" connected_to="lumi_link8"/>
 </robot>
 <!-- <asset>

Commit message: Added lumi_ee to fix error on rosrun

File: model/robots/hand.xacro (robot description, xacro)
@@ -62,4 +62,10 @@
       <mimic joint="${ns}_finger_joint1" />
     </joint>
+    <link name="lumi_ee"/>
+    <joint name="ee_fjoint" type="fixed">
+      <origin rpy="0 0 0" xyz="0 0 0.116"/>
+      <parent link="lumi_hand"/>
+      <child link="lumi_ee"/>
+    </joint>
   </xacro:macro>
 </robot>
