Commit message: fix handle

File: model/robots/robot_door.urdf.xacro (robot description, xacro)
@@ -49,4 +49,5 @@
         <origin xyz="0.052 -0.06 0.095" rpy="0 0 0"/>
         <limit lower="0" upper="${pi/6}" effort="10" velocity="10"/>
+        <axis xyz="0 1 0"/>
         <parent link="door"/>
         <child link="handle_core"/>

Commit message: scaled down stl meshes

File: model/robots/robot_door.urdf.xacro (robot description, xacro)
@@ -19,10 +19,10 @@
         <visual>
             <geometry>
-              <mesh scale="0.001 0.001 0.001" filename="package://franka_sim/model/meshes/door_v4_bin.stl"/>
-            </geometry>
-        </visual>
-       <collision>
-           <geometry>
-               <mesh scale="0.001 0.001 0.001" filename="package://franka_sim/model/meshes/door_v4_bin.stl"/>
+              <mesh filename="package://franka_sim/model/meshes/door_v5_bin.stl"/>
+            </geometry>
+        </visual>
+       <collision>
+           <geometry>
+               <mesh filename="package://franka_sim/model/meshes/door_v5_bin.stl"/>
            </geometry>
        </collision>
@@ -37,10 +37,10 @@
         <visual>
             <geometry>
-              <mesh scale="0.001 0.001 0.001" filename="package://franka_sim/model/meshes/handle_v4_core_bin.stl"/>
-            </geometry>
-        </visual>
-       <collision>
-           <geometry>
-               <mesh scale="0.001 0.001 0.001" filename="package://franka_sim/model/meshes/handle_v4_core_bin.stl"/>
+              <mesh filename="package://franka_sim/model/meshes/handle_v5_core_bin.stl"/>
+            </geometry>
+        </visual>
+       <collision>
+           <geometry>
+               <mesh filename="package://franka_sim/model/meshes/handle_v5_core_bin.stl"/>
            </geometry>
        </collision>
@@ -56,10 +56,10 @@
         <visual>
             <geometry>
-              <mesh scale="0.001 0.001 0.001" filename="package://franka_sim/model/meshes/handle_v4_beam_bin.stl"/>
-            </geometry>
-        </visual>
-       <collision>
-           <geometry>
-               <mesh scale="0.001 0.001 0.001" filename="package://franka_sim/model/meshes/handle_v4_beam_bin.stl"/>
+              <mesh filename="package://franka_sim/model/meshes/handle_v5_beam_bin.stl"/>
+            </geometry>
+        </visual>
+       <collision>
+           <geometry>
+               <mesh filename="package://franka_sim/model/meshes/handle_v5_beam_bin.stl"/>
            </geometry>
        </collision>
@@ -73,10 +73,10 @@
         <visual>
             <geometry>
-              <mesh scale="0.001 0.001 0.001" filename="package://franka_sim/model/meshes/handle_v4_latch_bin.stl"/>
-            </geometry>
-        </visual>
-       <collision>
-           <geometry>
-               <mesh scale="0.001 0.001 0.001" filename="package://franka_sim/model/meshes/handle_v4_latch_bin.stl"/>
+              <mesh filename="package://franka_sim/model/meshes/handle_v5_latch_bin.stl"/>
+            </geometry>
+        </visual>
+       <collision>
+           <geometry>
+               <mesh filename="package://franka_sim/model/meshes/handle_v5_latch_bin.stl"/>
            </geometry>
        </collision>
@@ -90,10 +90,10 @@
         <visual>
             <geometry>
-              <mesh scale="0.001 0.001 0.001" filename="package://franka_sim/model/meshes/frame_v4_leftpillar_back_bin.stl"/>
-            </geometry>
-        </visual>
-       <collision>
-           <geometry>
-               <mesh scale="0.001 0.001 0.001" filename="package://franka_sim/model/meshes/frame_v4_leftpillar_back_bin.stl"/>
+              <mesh filename="package://franka_sim/model/meshes/frame_v5_leftpillar_back_bin.stl"/>
+            </geometry>
+        </visual>
+       <collision>
+           <geometry>
+               <mesh filename="package://franka_sim/model/meshes/frame_v5_leftpillar_back_bin.stl"/>
            </geometry>
        </collision>
@@ -107,10 +107,10 @@
         <visual>
             <geometry>
-              <mesh scale="0.001 0.001 0.001" filename="package://franka_sim/model/meshes/frame_v4_leftpillar_front_bin.stl"/>
-            </geometry>
-        </visual>
-       <collision>
-           <geometry>
-               <mesh scale="0.001 0.001 0.001" filename="package://franka_sim/model/meshes/frame_v4_leftpillar_front_bin.stl"/>
+              <mesh filename="package://franka_sim/model/meshes/frame_v5_leftpillar_front_bin.stl"/>
+            </geometry>
+        </visual>
+       <collision>
+           <geometry>
+               <mesh filename="package://franka_sim/model/meshes/frame_v5_leftpillar_front_bin.stl"/>
            </geometry>
        </collision>
@@ -124,10 +124,10 @@
         <visual>
             <geometry>
-              <mesh scale="0.001 0.001 0.001" filename="package://franka_sim/model/meshes/frame_v4_rightpillar_bin.stl"/>
-            </geometry>
-        </visual>
-       <collision>
-           <geometry>
-               <mesh scale="0.001 0.001 0.001" filename="package://franka_sim/model/meshes/frame_v4_rightpillar_bin.stl"/>
+              <mesh filename="package://franka_sim/model/meshes/frame_v5_rightpillar_bin.stl"/>
+            </geometry>
+        </visual>
+       <collision>
+           <geometry>
+               <mesh filename="package://franka_sim/model/meshes/frame_v5_rightpillar_bin.stl"/>
            </geometry>
        </collision>
@@ -141,10 +141,10 @@
         <visual>
             <geometry>
-              <mesh scale="0.001 0.001 0.001" filename="package://franka_sim/model/meshes/frame_v4_top_bottom_bin.stl"/>
-            </geometry>
-        </visual>
-       <collision>
-           <geometry>
-               <mesh scale="0.001 0.001 0.001" filename="package://franka_sim/model/meshes/frame_v4_top_bottom_bin.stl"/>
+              <mesh filename="package://franka_sim/model/meshes/frame_v5_top_bottom_bin.stl"/>
+            </geometry>
+        </visual>
+       <collision>
+           <geometry>
+               <mesh filename="package://franka_sim/model/meshes/frame_v5_top_bottom_bin.stl"/>
            </geometry>
        </collision>
@@ -158,10 +158,10 @@
         <visual>
             <geometry>
-              <mesh scale="0.001 0.001 0.001" filename="package://franka_sim/model/meshes/frame_v4_top_bottom_bin.stl"/>
-            </geometry>
-        </visual>
-       <collision>
-           <geometry>
-               <mesh scale="0.001 0.001 0.001" filename="package://franka_sim/model/meshes/frame_v4_top_bottom_bin.stl"/>
+              <mesh filename="package://franka_sim/model/meshes/frame_v5_top_bottom_bin.stl"/>
+            </geometry>
+        </visual>
+       <collision>
+           <geometry>
+               <mesh filename="package://franka_sim/model/meshes/frame_v5_top_bottom_bin.stl"/>
            </geometry>
        </collision>
@@ -174,12 +174,12 @@
 </robot>
 <!-- <asset>
-        <mesh file="stl/frame_v4_leftpillar_back_bin.stl" name="frame_left"/>
-        <mesh file="stl/frame_v4_leftpillar_front_bin.stl" name="frame_left_front"/>
-        <mesh file="stl/frame_v4_rightpillar_bin.stl" name="frame_right"/>
-        <mesh file="stl/frame_v4_top_bottom_bin.stl" name="frame_top_bottom"/>
-        <mesh file="stl/door_v4_bin.stl" name="door"/>
-        <mesh file="stl/handle_v4_beam_bin.stl" name="handle_beam"/>
-        <mesh file="stl/handle_v4_latch_bin.stl" name="handle_latch"/>
-        <mesh file="stl/handle_v4_core_bin.stl" name="handle_core"/>
+        <mesh file="stl/frame_v5_leftpillar_back_bin.stl" name="frame_left"/>
+        <mesh file="stl/frame_v5_leftpillar_front_bin.stl" name="frame_left_front"/>
+        <mesh file="stl/frame_v5_rightpillar_bin.stl" name="frame_right"/>
+        <mesh file="stl/frame_v5_top_bottom_bin.stl" name="frame_top_bottom"/>
+        <mesh file="stl/door_v5_bin.stl" name="door"/>
+        <mesh file="stl/handle_v5_beam_bin.stl" name="handle_beam"/>
+        <mesh file="stl/handle_v5_latch_bin.stl" name="handle_latch"/>
+        <mesh file="stl/handle_v5_core_bin.stl" name="handle_core"/>
 </asset> -->
 <!-- <body pos="0 0 0">

Commit message: fixed door hinge rotation axis

File: model/robots/robot_door.urdf.xacro (robot description, xacro)
@@ -28,9 +28,17 @@
        </collision>
     </link>
+    <joint name="door_to_hinge" type="fixed">
+        <origin xyz="-0.257 -0.044 0.005" rpy="0 0 0"/>
+        <parent link="door_link"/>
+        <child link="door"/>
+    </joint>
+    <link name="door_link"/>
     <joint name="door_hinge" type="revolute">
-        <origin xyz="0.005 0.005 0.005" rpy="0 0 0"/>
+        <!-- <origin xyz="0.005 0.005 0.005" rpy="0 0 0"/> -->
+        <origin xyz="0.262 0.049 0" rpy="0 0 0"/>
         <limit lower="0" upper="${pi/2}" effort="10" velocity="10"/>
-        <parent link="door_base"/>
-        <child link="door"/>
+        <axis xyz="0 0 -1"/>
+        <parent link="door_base"/>
+        <child link="door_link"/>
     </joint>
     <link name="handle_core">

Commit message: Cleaned code

File: model/robots/robot_door.urdf.xacro (robot description, xacro)
@@ -7,12 +7,8 @@
     <mujoco>
         <compiler meshdir="../meshes/" balanceinertia="true" discardvisual="false"/>
-        <!--<option cone="elliptic" impratio="10">
-            <geom friction="1.5 0.005 0.0001" solimp="0.99 0.99 0.01" solref="0.01 1"/>
-        </option>-->
     </mujoco>
     <link name="base_link"/>
     <link name="door_base"/>
     <joint name="door_base_joint" type="fixed">
-        <!-- <origin xyz="0.0 0.0 0.052" rpy="0 0 ${pi}"/> -->
         <origin xyz="0.4 0.25 0.052" rpy="0 0 ${-pi/2}"/>
         <parent link="base_link"/>
@@ -38,5 +34,4 @@
     <link name="door_link"/>
     <joint name="door_hinge" type="revolute">
-        <!-- <origin xyz="0.005 0.005 0.005" rpy="0 0 0"/> -->
         <origin xyz="0.262 0.049 0" rpy="0 0 0"/>
         <limit lower="0" upper="${pi/2}" effort="10" velocity="10"/>

Commit message: added small collision box

File: model/robots/robot_door.urdf.xacro (robot description, xacro)
@@ -62,5 +62,5 @@
     <!-- TODO: replace collision with some "dummy" stl file which would not collide with robot -->
     <link name="handle_beam">
-        <!--<visual>
+        <visual>
             <geometry>
               <mesh filename="package://franka_sim/model/meshes/handle_v5_beam_bin.stl"/>
@@ -68,4 +68,9 @@
         </visual>
         <collision>
+            <geometry>
+                <box size="0.005 0.005 0.005"/>
+            </geometry>
+        </collision>
+        <!--<collision>
            <geometry>
                <mesh filename="package://franka_sim/model/meshes/handle_v5_beam_bin.stl"/>
