Commit message: changed hinges to revolutes, and added some changess made to urdf to xacro as well. The limits are not verified though.

File: model/robots/robot_door.urdf (robot description, URDF)
Before this commit: robot lumi, 23 links, 22 joints
Joints:
- joint door_hinge: limit (none) -> lower=0 upper=90 effort=10 velocity=10; type fixed -> revolute
- joint handle_core: limit (none) -> lower=0 upper=90 effort=10 velocity=10; type fixed -> revolute

File: model/robots/robot_door.urdf.xacro (robot description, xacro)
@@ -26,6 +26,7 @@
        </collision>
     </link>
-    <joint name="door_joint" type="fixed">
+    <joint name="door_hinge" type="revolute">
         <origin xyz="0.005 0.005 0.005" rpy="0 0 0"/>
+        <limit lower="0" upper="90" effort="10" velocity="10"/>
         <parent link="door_base"/>
         <child link="door"/>
@@ -43,6 +44,7 @@
        </collision>
     </link>
-    <joint name="handle_core_joint" type="fixed">
+    <joint name="handle_core" type="revolute">
         <origin xyz="0.052 -0.06 0.095" rpy="0 0 0"/>
+        <limit lower="0" upper="90" effort="10" velocity="10"/>
         <parent link="door"/>
         <child link="handle_core"/>

Commit message: test the pick and place

File: model/robots/robot_door.urdf (robot description, URDF)
Before this commit: robot lumi, 23 links, 22 joints
Joints:
- joint door_base_joint: origin xyz=0.0 0.0 0.0 rpy=0 0 0 -> xyz=0.4 0.25 0.052 rpy=0 0 -1.57079632679
- joint door_hinge: limit lower=0 upper=90 effort=10 velocity=10 -> lower=0 upper=1.57079632679 effort=10 velocity=10
- joint handle_core: limit lower=0 upper=90 effort=10 velocity=10 -> lower=0 upper=0.523598775598 effort=10 velocity=10
- joint lumi_joint_base_link: origin xyz=0.2 0.2 0.0 rpy=0 0 0 -> xyz=-0.4 0.15 0.0 rpy=0 0 0

Commit message: Robot turns handle

File: model/robots/robot_door.urdf (robot description, URDF)
Before this commit: robot lumi, 23 links, 22 joints
Links:
- added link door_link
- added link lumi_ee
- link door: geometry collision mesh filename=package://franka_sim/model/meshes/door_v5_bin.stl; visual mesh filename=package://franka_sim/model/meshes/door_v5_bin.stl
- link frame_bottom: geometry collision mesh filename=package://franka_sim/model/meshes/frame_v5_top_bottom_bin.s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; visual mesh filename=package://franka_sim/model/meshes/frame_v5_top_bottom_bin.s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
- link frame_left: geometry collision mesh filename=package://franka_sim/model/meshes/frame_v5_leftpillar_back_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; visual mesh filename=package://franka_sim/model/meshes/frame_v5_leftpillar_back_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
- link frame_left_front: geometry collision mesh filename=package://franka_sim/model/meshes/frame_v5_leftpillar_front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; visual mesh filename=package://franka_sim/model/meshes/frame_v5_leftpillar_front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
- link frame_right: geometry collision mesh filename=package://franka_sim/model/meshes/frame_v5_rightpillar_bin.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; visual mesh filename=package://franka_sim/model/meshes/frame_v5_rightpillar_bin.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
- link frame_top: geometry collision mesh filename=package://franka_sim/model/meshes/frame_v5_top_bottom_bin.s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; visual mesh filename=package://franka_sim/model/meshes/frame_v5_top_bottom_bin.s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
- link handle_beam: geometry 
- link handle_core: geometry collision mesh filename=package://franka_sim/model/meshes/handle_v5_core_bin.stl; visual mesh filename=package://franka_sim/model/meshes/handle_v5_core_bin.stl
- link handle_latch: geometry collision mesh filename=package://franka_sim/model/meshes/handle_v5_latch_bin.stl; visual mesh filename=package://franka_sim/model/meshes/handle_v5_latch_bin.stl
Joints:
- added joint door_to_hinge: type fixed, parent door_link, child door, origin xyz=-0.257 -0.044 0.005 rpy=0 0 0
- added joint ee_fjoint: type fixed, parent lumi_hand, child lumi_ee, origin xyz=0 0 0.116 rpy=0 0 0
- joint door_hinge: axis (none) -> 0 0 -1; child door -> door_link; origin xyz=0.005 0.005 0.005 rpy=0 0 0 -> xyz=0.262 0.049 0 rpy=0 0 0
- joint handle_core: axis (none) -> 0 1 0

File: model/robots/robot_door.urdf.xacro (robot description, xacro)
@@ -7,4 +7,7 @@
     <mujoco>
         <compiler meshdir="../meshes/" balanceinertia="true" discardvisual="false"/>
+        <!--<option cone="elliptic" impratio="10">
+            <geom friction="1.5 0.005 0.0001" solimp="0.99 0.99 0.01" solref="0.01 1"/>
+        </option>-->
     </mujoco>
     <link name="base_link"/>
@@ -61,15 +64,17 @@
         <child link="handle_core"/>
     </joint>
+    <!-- handle_beam visuals and collisions removed due to problems with moveit collisions between robot left/right fingers and handle_beam -->
+    <!-- TODO: replace collision with some "dummy" stl file which would not collide with robot -->
     <link name="handle_beam">
-        <visual>
+        <!--<visual>
             <geometry>
               <mesh filename="package://franka_sim/model/meshes/handle_v5_beam_bin.stl"/>
             </geometry>
         </visual>
-       <collision>
+        <collision>
            <geometry>
                <mesh filename="package://franka_sim/model/meshes/handle_v5_beam_bin.stl"/>
            </geometry>
-       </collision>
+        </collision>-->
     </link>
     <joint name="handle_beam_joint" type="fixed">

Commit message: Added comments and cleaned code

File: model/robots/robot_door.urdf (robot description, URDF)
Before this commit: robot lumi, 25 links, 24 joints
Links:
- link handle_beam: geometry collision box size=0.005 0.005 0.005; visual mesh filename=package://franka_sim/model/meshes/handle_v5_beam_bin.stl

File: model/robots/robot_door.urdf.xacro (robot description, xacro)
@@ -15,21 +15,4 @@
         <child link="door_base"/>
     </joint>
-    <link name="door">
-        <visual>
-            <geometry>
-              <mesh filename="package://franka_sim/model/meshes/door_v5_bin.stl"/>
-            </geometry>
-        </visual>
-       <collision>
-           <geometry>
-               <mesh filename="package://franka_sim/model/meshes/door_v5_bin.stl"/>
-           </geometry>
-       </collision>
-    </link>
-    <joint name="door_to_hinge" type="fixed">
-        <origin xyz="-0.257 -0.044 0.005" rpy="0 0 0"/>
-        <parent link="door_link"/>
-        <child link="door"/>
-    </joint>
     <link name="door_link"/>
     <joint name="door_hinge" type="revolute">
@@ -39,4 +22,21 @@
         <parent link="door_base"/>
         <child link="door_link"/>
+    </joint>
+    <link name="door">
+        <visual>
+            <geometry>
+              <mesh filename="package://franka_sim/model/meshes/door_v5_bin.stl"/>
+            </geometry>
+        </visual>
+       <collision>
+           <geometry>
+               <mesh filename="package://franka_sim/model/meshes/door_v5_bin.stl"/>
+           </geometry>
+       </collision>
+    </link>
+    <joint name="door_to_hinge" type="fixed">
+        <origin xyz="-0.257 -0.044 0.005" rpy="0 0 0"/>
+        <parent link="door_link"/>
+        <child link="door"/>
     </joint>
     <link name="handle_core">
@@ -59,6 +59,5 @@
         <child link="handle_core"/>
     </joint>
-    <!-- handle_beam visuals and collisions removed due to problems with moveit collisions between robot left/right fingers and handle_beam -->
-    <!-- TODO: replace collision with some "dummy" stl file which would not collide with robot -->
+    <!-- handle_beam collision mesh replaced by dummy due to issues with moveit collisions between robot left/right fingers and handle_beam -->
     <link name="handle_beam">
         <visual>
